File: kicad/onboarding-electrical-josh/onboarding-electrical-josh.kicad_sch (KiCad schematic)
At the start: 0 parts

Commit message: implemented boost converter schematic
Parts:
- added C1: 330, symbol Device:C
- added C2: 100, symbol Device:C
- added C3: 1500, symbol Device:C
- added D1: D_Schottky, symbol Device:D_Schottky
- added L1: L, symbol Device:L
- added R1: .22, symbol Device:R
- added R2: 180, symbol Device:R
- added R3: 2200, symbol Device:R
- added R4: 40040, symbol Device:R
- added U1: MC33063AP, Package_DIP:DIP-8_W7.62mm, symbol Regulator_Switching:MC33063AP
Connections:
- new net: C1.1, D1.1 (K)
- new net: D1.2 (A), L1.2, U1.1 (SwC)
- new net: L1.1, R1.2, R2.2, U1.7 (Ipk)
- new net: R3.1, U1.5 (Vfb)
- new net: R2.1, U1.8 (DC)
- new net: C3.2, U1.3 (TC)
- new net Vin: C2.2, R1.1, U1.6 (Vin)
- new net Vout: C1.2, C2.1, C3.1, R3.2, R4.1, R4.2, U1.2 (SwE), U1.4 (GND)

Commit message: fixed wiring issues
Connections:
- net Vout: now also C1.1, D1.1 (K); no longer C1.2, C2.1, C3.1, R3.2, R4.1, U1.2 (SwE), U1.4 (GND)
- new net GND: C1.2, C2.1, C3.1, R3.2, R4.1, U1.2 (SwE), U1.4 (GND)
